File: pcb/rpi-gardener-hat.kicad_pcb (KiCad board)
At the start: 2 copper layers, 65 x 56 mm, 13 parts, among them J1 RPi_GPIO, J2 OLED_RPi, J3 LCD_I2C, J4 DHT22, J5 OLED_Pico, J6 MOISTURE_1, J7 MOISTURE_2, J8 MOISTURE_3, U1 Pico

Commit message: WIP
Parts:
- H1, H2, H3, H4: footprint MountingHole:MountingHole_2.7mm_M2.5 -> MountingHole:MountingHole_3.2mm_M3
- J1: moved to B.Cu
- moved U1 88.5 mm to (120.0, 83.0)
- moved J4 82.3 mm to (95.0, 94.0)
- moved J3 81.7 mm to (95.0, 82.0)
- moved J2 81.1 mm to (95.0, 70.0)
- moved J6 80.2 mm to (105.0, 82.0)
- moved J7 80.2 mm to (105.0, 91.0)
- moved J8 80.2 mm to (105.0, 100.0)
- moved J5 79.5 mm to (105.0, 70.0)
- moved J1 76.0 mm to (85.4, 57.8), turned to 270 degrees
- moved H3 75.7 mm to (80.5, 108.5)
- moved H4 75.7 mm to (138.5, 108.5)
- moved H1 75.4 mm to (80.5, 59.0)
- moved H2 75.4 mm to (138.5, 59.0)
Other:
- board size 65 x 56 mm -> 65 x 56.5 mm
- rule pad_to_mask_clearance: 0 -> 0.051

Commit message: Updated
Parts:
- J6: renamed from J8; value MOISTURE_3 -> MOIST1
- J7: value MOISTURE_2 -> MOIST2
- J8: renamed from J6; value MOISTURE_1 -> MOIST3
- moved U1 34.1 mm to (87.4, 93.1), turned to 90 degrees
- moved J6 31.9 mm to (114.5, 69.5)
- moved J5 28.0 mm to (133.0, 69.5)
- moved J4 26.7 mm to (105.5, 69.5)
- moved J7 26.2 mm to (120.0, 69.5)
- moved J8 24.0 mm to (125.5, 69.5)
- moved J3 15.0 mm to (95.5, 67.0)
- moved J2 7.16 mm to (88.5, 67.0)
Other:
- board text added: "RPi Gardener HAT v1.2 github.com/smallwat3r/rpi-gardener"
- board text removed: "RPi Gardener HAT v1.2"

Commit message: Fix
Connections:
- J5 pad 2: PICO_GND -> GND
- J6 pad 3: PICO_GND -> GND
- J7 pad 3: PICO_GND -> GND
- J8 pad 3: PICO_GND -> GND
- U1 pad 13: PICO_GND -> GND
- U1 pad 18: PICO_GND -> GND
- U1 pad 23: PICO_GND -> GND
- U1 pad 28: PICO_GND -> GND
- U1 pad 3: PICO_GND -> GND
- U1 pad 33: PICO_GND -> GND
- U1 pad 38: PICO_GND -> GND
- U1 pad 8: PICO_GND -> GND
Routing:
- added copper zone on B.Cu, net GND
- added copper zone on F.Cu, net GND

Commit message: Add gerber file
Parts:
- moved J6 5.59 mm to (109.5, 67.0)
- moved J7 4.30 mm to (116.5, 67.0)
- moved J4 3.91 mm to (102.5, 67.0)
- moved J5 3.54 mm to (130.5, 67.0)
- moved J8 3.20 mm to (123.5, 67.0)
Routing:
- net GP0_SDA: track 0.00 -> 60.3 mm
- net GP1_SCL: track 0.00 -> 55.5 mm
- net PICO_3V3: track 0.00 -> 43.7 mm
- net I2C_SCL: track 0.00 -> 26.0 mm
- net I2C_SDA: track 0.00 -> 23.6 mm
- net GP26_ADC0: track 0.00 -> 20.1 mm
- net GP27_ADC1: track 0.00 -> 18.3 mm
- net GP28_ADC2: track 0.00 -> 18.2 mm
- net +3V3: track 0.00 -> 15.9 mm
- net +5V: track 0.00 -> 12.3 mm
- net GPIO17_DHT: track 0.00 -> 11.0 mm
